File: Xiaomi2Ali-Smart-Plug-WIFI-Module.sch (KiCad schematic (older format))
At the start: 7 parts, among them J1 Conn_01x07, J2 Conn_01x03, SW1 SW_Push

Commit message: Updated: 2019-02-17 20:07:23
Parts:
- D1: value LED -> LED_blue
- D2: value LED -> LED_yellow
- R1, R2: value R -> 1K
Changed lines of the file:
@@
 P 5450 3750
 F 0 "R1" V 5243 3750 50  0000 C CNN
-F 1 "R" V 5334 3750 50  0000 C CNN
+F 1 "1K" V 5334 3750 50  0000 C CNN
 F 2 "Resistor_SMD:R_1206_3216Metric" V 5380 3750 50  0001 C CNN
 F 3 "~" H 5450 3750 50  0001 C CNN
@@
 P 5450 4100
 F 0 "R2" V 5243 4100 50  0000 C CNN
-F 1 "R" V 5334 4100 50  0000 C CNN
+F 1 "1K" V 5334 4100 50  0000 C CNN
 F 2 "Resistor_SMD:R_1206_3216Metric" V 5380 4100 50  0001 C CNN
 F 3 "~" H 5450 4100 50  0001 C CNN
@@
 P 5050 3750
 F 0 "D1" H 5042 3495 50  0000 C CNN
-F 1 "LED" H 5042 3586 50  0000 C CNN
+F 1 "LED_blue" H 5042 3586 50  0000 C CNN
 F 2 "LED_SMD:LED_1206_3216Metric" H 5050 3750 50  0001 C CNN
 F 3 "~" H 5050 3750 50  0001 C CNN
@@
 P 5050 4100
 F 0 "D2" H 5042 3845 50  0000 C CNN
-F 1 "LED" H 5042 3936 50  0000 C CNN
+F 1 "LED_yellow" H 5042 3936 50  0000 C CNN
 F 2 "LED_SMD:LED_1206_3216Metric" H 5050 4100 50  0001 C CNN
 F 3 "~" H 5050 4100 50  0001 C CNN

Commit message: Updated: 2019-02-20 16:21:37
Parts:
- SW1: footprint Button_Switch_SMD:SW_SPST_TL3305A -> Button_Switch_SMD:SW_SPST_B3S-1000
Changed lines of the file:
@@
 F 0 "SW1" H 5400 3635 50  0000 C CNN
 F 1 "SW_Push" H 5400 3544 50  0000 C CNN
-F 2 "Button_Switch_SMD:SW_SPST_TL3305A" H 5400 3550 50  0001 C CNN
+F 2 "Button_Switch_SMD:SW_SPST_B3S-1000" H 5400 3550 50  0001 C CNN
 F 3 "" H 5400 3550 50  0001 C CNN
 	1    5400 3350
